File: DextraBoard.kicad_pcb (KiCad board)
At the start: 4 copper layers, 73 x 33 mm, 32 parts, among them J1 Conn_02x07_Counter_Clockwise, J2 Conn_02x07_Counter_Clockwise, J3 Conn_02x07_Counter_Clockwise, J4 Conn_02x06_Counter_Clockwise, J5 Conn_02x07_Counter_Clockwise, J6 USB_C_Receptacle_USB2.0, J7 Conn_02x07_Counter_Clockwise, J9 USB_C_Receptacle_USB2.0, SW1 SW_SPDT, SW2 SW_SPDT, U2 ESP32-PICO-D4, U3 N76E003AQ20, U4 N76E003AQ20, U5 N76E003AQ20, U6 N76E003AQ20, U7 MCP73811T-420I-OT, U8 CH340E

Commit message: redesigned everything x)
new BMS design, switched to ESP32-S3 with external antenna, implement USB-C PD, add analog mux, add PWM controller, add USB to serial
Parts:
- removed TP1, TP2, TP3, TP4, TP5, TP6: TestPoint, TestPoint:TestPoint_Pad_D1.5mm
- removed U5: N76E003AQ20, Footprint:QFN40P300X300X80-21N
- added C1: 0.1uF, Capacitor_SMD:C_0402_1005Metric, B.Cu at (61.9, 30.4)
- added C2: 0.1uF, Capacitor_SMD:C_0402_1005Metric, B.Cu at (61.9, 32.4)
- added C3: 0.1uF, Capacitor_SMD:C_0402_1005Metric, B.Cu at (85.4, 22.5)
- added C4: 0.1uF, Capacitor_SMD:C_0402_1005Metric, B.Cu at (97.3, 33.3)
- added C5: 0.1uF, Capacitor_SMD:CP_Elec_4x3, B.Cu at (102.6, 32.2)
- added C6: 0.1uF, Capacitor_SMD:CP_Elec_4x3, B.Cu at (90.7, 24.4)
- added D1: LED, LED_SMD:LED_0805_2012Metric, B.Cu at (96.5, 30.8)
- added J8: Conn_01x03_Female, Connector_JST:JST_XH_B3B-XH-A_1x03_P2.50mm_Vertical, F.Cu at (108.4, 77.2)
- added Q1: HX2300A, Package_TO_SOT_SMD:SOT-23, B.Cu at (72.0, 75.9)
- added Q2: HX2300A, Package_TO_SOT_SMD:SOT-23, B.Cu at (78.0, 75.9)
- added Q4: HX2300A, Package_TO_SOT_SMD:SOT-23, B.Cu at (81.9, 71.9)
- added Q6: HX2300A, Package_TO_SOT_SMD:SOT-23, B.Cu at (85.9, 71.9)
- added R10: 10K, Resistor_SMD:R_0201_0603Metric, B.Cu at (59.2, 30.3)
- added R11: 1K, Resistor_SMD:R_0201_0603Metric, B.Cu at (93.3, 28.2)
- added R12: 1K, Resistor_SMD:R_0201_0603Metric, B.Cu at (85.6, 24.3)
- added R13: R, Resistor_SMD:R_0201_0603Metric, B.Cu at (90.9, 28.2)
- added R14: 2K, Resistor_SMD:R_0201_0603Metric, B.Cu at (90.6, 30.0)
- added R15: 330R, Resistor_SMD:R_0201_0603Metric, B.Cu at (88.4, 28.2)
- added R16: 330R, Resistor_SMD:R_0201_0603Metric, B.Cu at (85.6, 26.1)
- added U1: ESP32-S3-WROOM-1, Espressif:ESP32-S3-WROOM-1U, B.Cu at (100.1, 63.5)
- R1, R2: value 10K -> 100R; moved to B.Cu
- R7, R9: moved to B.Cu
- R8: value 1M -> 2M; moved to B.Cu
- U2: value ESP32-PICO-D4 -> PCA9685PW; footprint Package_DFN_QFN:QFN-48-1EP_7x7mm_P0.5mm_EP5.3x5.3mm -> Package_SO:TSSOP-28_4.4x9.7mm_P0.65mm; moved to B.Cu
- U3, U4: value N76E003AQ20 -> CD74HC4067SM; footprint Footprint:QFN40P300X300X80-21N -> Package_SO:SSOP-24_5.3x8.2mm_P0.65mm; moved to B.Cu
- U6: value N76E003AQ20 -> HY2213; footprint Footprint:QFN40P300X300X80-21N -> Package_TO_SOT_SMD:SOT-23-6; moved to B.Cu
- U7: value MCP73811T-420I-OT -> HY2213; footprint Package_TO_SOT_SMD:SOT-23-5 -> Package_TO_SOT_SMD:SOT-23-6; moved to B.Cu
- U8: value CH340E -> HY2120; footprint Package_SO:MSOP-10_3x3mm_P0.5mm -> Package_TO_SOT_SMD:SOT-23-6; moved to B.Cu
- moved R2 55.3 mm to (82.7, 22.4), turned to 180 degrees
- moved R1 45.3 mm to (93.1, 31.7), turned to 180 degrees
- moved U2 38.9 mm to (71.0, 53.0), turned to 180 degrees
- moved R9 32.1 mm to (73.4, 24.8), turned to 0 degrees
- moved R8 30.0 mm to (75.4, 24.8), turned to 180 degrees
- moved R7 23.5 mm to (93.1, 30.0), turned to 180 degrees
- moved U7 23.2 mm to (78.0, 71.9)
- moved U3 13.9 mm to (61.5, 63.1), turned to 180 degrees
- moved U8 11.1 mm to (85.9, 76.9), turned to -90 degrees
- moved U6 9.26 mm to (71.9, 71.9), turned to 180 degrees
- moved J4 8.90 mm to (105.6, 63.5)
- moved U4 3.80 mm to (82.3, 53.1)
Connections:
- J1 pad 10: /N76E003s (PWM + ADC + IO)/ANA0_4 -> /N76E003s (PWM + ADC + IO)/MUX_CH4
- J1 pad 11: /N76E003s (PWM + ADC + IO)/ANA0_3 -> /N76E003s (PWM + ADC + IO)/MUX_CH3
- J1 pad 12: /N76E003s (PWM + ADC + IO)/ANA0_2 -> /N76E003s (PWM + ADC + IO)/MUX_CH2
- J1 pad 13: /N76E003s (PWM + ADC + IO)/ANA0_1 -> /N76E003s (PWM + ADC + IO)/MUX_CH1
- J1 pad 14: /N76E003s (PWM + ADC + IO)/ANA0_0 -> /N76E003s (PWM + ADC + IO)/MUX_CH0
- J1 pad 2: /N76E003s (PWM + ADC + IO)/PWM0_0 -> /N76E003s (PWM + ADC + IO)/PWM14
- J1 pad 3: /N76E003s (PWM + ADC + IO)/PWM0_1 -> /N76E003s (PWM + ADC + IO)/PWM15
- J1 pad 4: /N76E003s (PWM + ADC + IO)/PWM0_2 -> /N76E003s (PWM + ADC + IO)/PWM4
- J1 pad 5: /N76E003s (PWM + ADC + IO)/PWM0_3 -> /N76E003s (PWM + ADC + IO)/PWM5
- J1 pad 6: /N76E003s (PWM + ADC + IO)/RXD0 -> /N76E003s (PWM + ADC + IO)/IO9
- J1 pad 9: /N76E003s (PWM + ADC + IO)/ANA0_5 -> /N76E003s (PWM + ADC + IO)/MUX_CH5
- J2 pad 10: /N76E003s (PWM + ADC + IO)/ANA1_3 -> /N76E003s (PWM + ADC + IO)/MUX_CH10
- J2 pad 11: /N76E003s (PWM + ADC + IO)/ANA1_2 -> /N76E003s (PWM + ADC + IO)/MUX_CH9
- J2 pad 12: /N76E003s (PWM + ADC + IO)/ANA1_1 -> /N76E003s (PWM + ADC + IO)/MUX_CH8
- J2 pad 13: /N76E003s (PWM + ADC + IO)/ANA1_0 -> /N76E003s (PWM + ADC + IO)/MUX_CH7
- J2 pad 14: /N76E003s (PWM + ADC + IO)/ANA0_6 -> /N76E003s (PWM + ADC + IO)/MUX_CH6
- J2 pad 2: /N76E003s (PWM + ADC + IO)/PWM0_4 -> /N76E003s (PWM + ADC + IO)/PWM10
- J2 pad 3: /N76E003s (PWM + ADC + IO)/PWM0_5 -> /N76E003s (PWM + ADC + IO)/PWM11
- J2 pad 4: /N76E003s (PWM + ADC + IO)/PWM1_0 -> /N76E003s (PWM + ADC + IO)/PWM12
- J2 pad 5: /N76E003s (PWM + ADC + IO)/PWM1_1 -> /N76E003s (PWM + ADC + IO)/PWM13
- J2 pad 6: /N76E003s (PWM + ADC + IO)/TXD0 -> /N76E003s (PWM + ADC + IO)/IO8
- J2 pad 9: /N76E003s (PWM + ADC + IO)/ANA1_4 -> /N76E003s (PWM + ADC + IO)/MUX_CH11
- J3 pad 10: /N76E003s (PWM + ADC + IO)/ANA2_2 -> /N76E003s (PWM + ADC + IO)/MUX_CH16
- J3 pad 11: /N76E003s (PWM + ADC + IO)/ANA2_1 -> /N76E003s (PWM + ADC + IO)/MUX_CH15
- J3 pad 12: /N76E003s (PWM + ADC + IO)/ANA2_0 -> /N76E003s (PWM + ADC + IO)/MUX_CH14
- J3 pad 13: /N76E003s (PWM + ADC + IO)/ANA1_6 -> /N76E003s (PWM + ADC + IO)/MUX_CH13
- J3 pad 14: /N76E003s (PWM + ADC + IO)/ANA1_5 -> /N76E003s (PWM + ADC + IO)/MUX_CH12
- J3 pad 2: /N76E003s (PWM + ADC + IO)/PWM1_2 -> /N76E003s (PWM + ADC + IO)/PWM6
- J3 pad 3: /N76E003s (PWM + ADC + IO)/PWM1_3 -> /N76E003s (PWM + ADC + IO)/PWM7
- J3 pad 4: /N76E003s (PWM + ADC + IO)/PWM1_4 -> /N76E003s (PWM + ADC + IO)/PWM8
- J3 pad 5: /N76E003s (PWM + ADC + IO)/PWM1_5 -> /N76E003s (PWM + ADC + IO)/PWM9
- J3 pad 6: /N76E003s (PWM + ADC + IO)/RXD1 -> /N76E003s (PWM + ADC + IO)/IO7
- J3 pad 9: /N76E003s (PWM + ADC + IO)/ANA2_3 -> /N76E003s (PWM + ADC + IO)/MUX_CH17
- J4 pad 10: /ANA2 -> /ANA0
- J4 pad 11: /N76E003s (PWM + ADC + IO)/TXD3 -> /IO15
- J4 pad 12: /N76E003s (PWM + ADC + IO)/TXD3 -> /IO13
- J4 pad 5: /N76E003s (PWM + ADC + IO)/TXD2 -> /N76E003s (PWM + ADC + IO)/IO4
- J4 pad 6: /N76E003s (PWM + ADC + IO)/RXD3 -> /IO14
- J4 pad 8: /ANA4 -> /ANA2
- J4 pad 9: /ANA3 -> /ANA1
- J5 pad 10: /N76E003s (PWM + ADC + IO)/ANA3_1 -> /N76E003s (PWM + ADC + IO)/MUX_CH22
- J5 pad 11: /N76E003s (PWM + ADC + IO)/ANA3_0 -> /N76E003s (PWM + ADC + IO)/MUX_CH21
- J5 pad 12: /N76E003s (PWM + ADC + IO)/ANA2_6 -> /N76E003s (PWM + ADC + IO)/MUX_CH20
- J5 pad 13: /N76E003s (PWM + ADC + IO)/ANA2_5 -> /N76E003s (PWM + ADC + IO)/MUX_CH19
- J5 pad 14: /N76E003s (PWM + ADC + IO)/ANA2_4 -> /N76E003s (PWM + ADC + IO)/MUX_CH18
- J5 pad 2: /N76E003s (PWM + ADC + IO)/PWM2_0 -> /PWM2
- J5 pad 3: /N76E003s (PWM + ADC + IO)/PWM2_1 -> /PWM3
- J5 pad 4: /N76E003s (PWM + ADC + IO)/PWM2_2 -> /N76E003s (PWM + ADC + IO)/PWM4
- J5 pad 5: /N76E003s (PWM + ADC + IO)/PWM2_3 -> /N76E003s (PWM + ADC + IO)/PWM5
- J5 pad 6: /N76E003s (PWM + ADC + IO)/TXD1 -> /N76E003s (PWM + ADC + IO)/IO6
- J5 pad 9: /N76E003s (PWM + ADC + IO)/ANA3_2 -> /N76E003s (PWM + ADC + IO)/MUX_CH23
- J7 pad 10: /ANA0 -> /N76E003s (PWM + ADC + IO)/MUX_CH28
- J7 pad 11: /N76E003s (PWM + ADC + IO)/ANA3_6 -> /N76E003s (PWM + ADC + IO)/MUX_CH27
- J7 pad 12: /N76E003s (PWM + ADC + IO)/ANA3_5 -> /N76E003s (PWM + ADC + IO)/MUX_CH26
- J7 pad 13: /N76E003s (PWM + ADC + IO)/ANA3_4 -> /N76E003s (PWM + ADC + IO)/MUX_CH25
- J7 pad 14: /N76E003s (PWM + ADC + IO)/ANA3_3 -> /N76E003s (PWM + ADC + IO)/MUX_CH24
- J7 pad 2: /N76E003s (PWM + ADC + IO)/PWM2_4 -> /PWM0
- J7 pad 3: /N76E003s (PWM + ADC + IO)/PWM2_5 -> /PWM1
- J7 pad 4: /N76E003s (PWM + ADC + IO)/PWM3_0 -> /PWM3
- J7 pad 5: /N76E003s (PWM + ADC + IO)/PWM3_1 -> /PWM2
- J7 pad 6: /N76E003s (PWM + ADC + IO)/RXD2 -> /N76E003s (PWM + ADC + IO)/IO5
- J7 pad 9: /ANA1 -> /N76E003s (PWM + ADC + IO)/MUX_CH29
- R1 pad 1: +3V3 -> +BATT
- R1 pad 2: /I2C_SDA -> Net-(R1-Pad2)
- R2 pad 1: +3V3 -> /MID_BAT
- R2 pad 2: /I2C_SCL -> Net-(R2-Pad2)
- R7 pad 1: GND -> Net-(R7-Pad1)
- R7 pad 2: Net-(R7-Pad2) -> GND
- U2 pad 1: Net-(U2-Pad1) -> unconnected-(U2-Pad1)
- U2 pad 10: /ANA1 -> /N76E003s (PWM + ADC + IO)/PWM4
- U2 pad 11: /ANA2 -> /N76E003s (PWM + ADC + IO)/PWM5
- U2 pad 12: /VSENSE -> /N76E003s (PWM + ADC + IO)/PWM6
- U2 pad 13: /ANA0 -> /N76E003s (PWM + ADC + IO)/PWM7
- U2 pad 14: unconnected-(U2-Pad14) -> GND
- U2 pad 15: /ANA3 -> /N76E003s (PWM + ADC + IO)/PWM8
- U2 pad 16: /ANA4 -> /N76E003s (PWM + ADC + IO)/PWM9
- U2 pad 17: unconnected-(U2-Pad17) -> /N76E003s (PWM + ADC + IO)/PWM10
- U2 pad 18: unconnected-(U2-Pad18) -> /N76E003s (PWM + ADC + IO)/PWM11
- U2 pad 19: unconnected-(U2-Pad19) -> /N76E003s (PWM + ADC + IO)/PWM12
- U2 pad 20: unconnected-(U2-Pad20) -> /N76E003s (PWM + ADC + IO)/PWM13
- U2 pad 21: unconnected-(U2-Pad21) -> /N76E003s (PWM + ADC + IO)/PWM14
- U2 pad 22: unconnected-(U2-Pad22) -> /N76E003s (PWM + ADC + IO)/PWM15
- U2 pad 26: unconnected-(U2-Pad26) -> /N76E003s (PWM + ADC + IO)/I2C_SCL
- U2 pad 27: unconnected-(U2-Pad27) -> /N76E003s (PWM + ADC + IO)/I2C_SDA
- U2 pad 28: unconnected-(U2-Pad28) -> +3.3V
- U2 pad 3: +3V3 -> unconnected-(U2-Pad3)
- U2 pad 4: +3V3 -> unconnected-(U2-Pad4)
- U2 pad 6: unconnected-(U2-Pad6) -> /PWM0
- U2 pad 7: unconnected-(U2-Pad7) -> /PWM1
- U2 pad 8: unconnected-(U2-Pad8) -> /PWM2
- U2 pad 9: unconnected-(U2-Pad9) -> /PWM3
- U3 pad 1: /N76E003s (PWM + ADC + IO)/ANA0_2 -> /ANA3
- U3 pad 10: /I2C_SDA -> /IO7
- U3 pad 11: /I2C_SCL -> /IO8
- U3 pad 12: /N76E003s (PWM + ADC + IO)/PWM0_3 -> GND
- U3 pad 13: /N76E003s (PWM + ADC + IO)/PWM0_4 -> /IO10
- U3 pad 14: /N76E003s (PWM + ADC + IO)/RXD0 -> /IO9
- U3 pad 15: /N76E003s (PWM + ADC + IO)/ANA0_6 -> GND
- U3 pad 16: /N76E003s (PWM + ADC + IO)/ANA0_5 -> /N76E003s (PWM + ADC + IO)/MUX_CH15
- U3 pad 17: /N76E003s (PWM + ADC + IO)/ANA0_1 -> /N76E003s (PWM + ADC + IO)/MUX_CH14
- U3 pad 18: Net-(TP3-Pad1) -> /N76E003s (PWM + ADC + IO)/MUX_CH13
- U3 pad 19: /N76E003s (PWM + ADC + IO)/ANA0_3 -> /N76E003s (PWM + ADC + IO)/MUX_CH12
- U3 pad 2: /N76E003s (PWM + ADC + IO)/ANA0_0 -> /N76E003s (PWM + ADC + IO)/MUX_CH7
- U3 pad 20: /N76E003s (PWM + ADC + IO)/ANA0_4 -> /N76E003s (PWM + ADC + IO)/MUX_CH11
- U3 pad 21: GND -> /N76E003s (PWM + ADC + IO)/MUX_CH10
- U3 pad 3: GND -> /N76E003s (PWM + ADC + IO)/MUX_CH6
- U3 pad 4: /N76E003s (PWM + ADC + IO)/TXD0 -> /N76E003s (PWM + ADC + IO)/MUX_CH5
- U3 pad 5: +3V3 -> /N76E003s (PWM + ADC + IO)/MUX_CH4
- U3 pad 6: /N76E003s (PWM + ADC + IO)/PWM0_5 -> /N76E003s (PWM + ADC + IO)/MUX_CH3
- U3 pad 7: /N76E003s (PWM + ADC + IO)/PWM0_2 -> /N76E003s (PWM + ADC + IO)/MUX_CH2
- U3 pad 8: /N76E003s (PWM + ADC + IO)/PWM0_1 -> /N76E003s (PWM + ADC + IO)/MUX_CH1
- U3 pad 9: /N76E003s (PWM + ADC + IO)/PWM0_0 -> /N76E003s (PWM + ADC + IO)/MUX_CH0
- U4 pad 1: /N76E003s (PWM + ADC + IO)/ANA1_2 -> /ANA4
- U4 pad 10: /I2C_SDA -> /IO7
- U4 pad 11: /I2C_SCL -> /IO8
- U4 pad 12: /N76E003s (PWM + ADC + IO)/PWM1_3 -> GND
- U4 pad 13: /N76E003s (PWM + ADC + IO)/PWM1_4 -> /IO10
- U4 pad 14: /N76E003s (PWM + ADC + IO)/RXD1 -> /IO9
- U4 pad 15: /N76E003s (PWM + ADC + IO)/ANA1_6 -> GND
- U4 pad 16: /N76E003s (PWM + ADC + IO)/ANA1_5 -> /N76E003s (PWM + ADC + IO)/MUX_CH31
- U4 pad 17: /N76E003s (PWM + ADC + IO)/ANA1_1 -> /N76E003s (PWM + ADC + IO)/MUX_CH30
- U4 pad 18: Net-(TP4-Pad1) -> /N76E003s (PWM + ADC + IO)/MUX_CH29
- U4 pad 19: /N76E003s (PWM + ADC + IO)/ANA1_3 -> /N76E003s (PWM + ADC + IO)/MUX_CH28
- U4 pad 2: /N76E003s (PWM + ADC + IO)/ANA1_0 -> /N76E003s (PWM + ADC + IO)/MUX_CH23
- U4 pad 20: /N76E003s (PWM + ADC + IO)/ANA1_4 -> /N76E003s (PWM + ADC + IO)/MUX_CH27
- U4 pad 21: GND -> /N76E003s (PWM + ADC + IO)/MUX_CH26
- U4 pad 3: GND -> /N76E003s (PWM + ADC + IO)/MUX_CH22
- U4 pad 4: /N76E003s (PWM + ADC + IO)/TXD1 -> /N76E003s (PWM + ADC + IO)/MUX_CH21
- U4 pad 5: +3V3 -> /N76E003s (PWM + ADC + IO)/MUX_CH20
- U4 pad 6: /N76E003s (PWM + ADC + IO)/PWM1_5 -> /N76E003s (PWM + ADC + IO)/MUX_CH19
- U4 pad 7: /N76E003s (PWM + ADC + IO)/PWM1_2 -> /N76E003s (PWM + ADC + IO)/MUX_CH18
- U4 pad 8: /N76E003s (PWM + ADC + IO)/PWM1_1 -> /N76E003s (PWM + ADC + IO)/MUX_CH17
- U4 pad 9: /N76E003s (PWM + ADC + IO)/PWM1_0 -> /N76E003s (PWM + ADC + IO)/MUX_CH16
- U6 pad 1: /N76E003s (PWM + ADC + IO)/ANA3_2 -> unconnected-(U6-Pad1)
- U6 pad 2: /N76E003s (PWM + ADC + IO)/ANA3_0 -> Net-(R1-Pad2)
- U6 pad 3: GND -> /MID_BAT
- U6 pad 4: /N76E003s (PWM + ADC + IO)/TXD3 -> unconnected-(U6-Pad4)
- U6 pad 5: +3V3 -> unconnected-(U6-Pad5)
- U6 pad 6: /N76E003s (PWM + ADC + IO)/PWM3_5 -> Net-(Q1-Pad1)
- U7 pad 2: GND -> Net-(R2-Pad2)
- U7 pad 3: +BATT -> -BATT
- U7 pad 4: VBUS -> unconnected-(U7-Pad4)
- U7 pad 5: Net-(R7-Pad2) -> unconnected-(U7-Pad5)
- U8 pad 1: /USB_DP -> /OD
- U8 pad 2: /USB_DN -> /OC
- U8 pad 3: GND -> Net-(R14-Pad2)
- U8 pad 4: unconnected-(U8-Pad4) -> Net-(C6-Pad1)
- U8 pad 5: unconnected-(U8-Pad5) -> /HY_VDD
- U8 pad 6: unconnected-(U8-Pad6) -> -BATT
Routing:
- net +3V3: track 177.0 -> 0.00 mm, vias 5 -> 0
- net /I2C_SDA: track 94.4 -> 0.00 mm, vias 5 -> 0
- net VBUS: track 90.5 -> 0.00 mm
- net /USB_DP: track 85.0 -> 0.00 mm, vias 1 -> 0
- net /I2C_SCL: track 78.2 -> 0.00 mm, vias 3 -> 0
- net +5V: track 75.6 -> 0.00 mm, vias 3 -> 0
- net /N76E003s (PWM + ADC + IO)/RXD0: track 75.2 -> 0.00 mm, vias 2 -> 0
- net /USB_DN: track 72.3 -> 0.00 mm, vias 1 -> 0
- net +BATT: track 67.2 -> 0.00 mm, vias 1 -> 0
- net /N76E003s (PWM + ADC + IO)/TXD2: track 63.8 -> 0.00 mm, vias 2 -> 0
- net /N76E003s (PWM + ADC + IO)/ANA0_0: track 47.3 -> 0.00 mm
- net /VSENSE: track 45.4 -> 0.00 mm, vias 2 -> 0
- net /N76E003s (PWM + ADC + IO)/PWM3_0: track 44.7 -> 0.00 mm, vias 2 -> 0
- net /N76E003s (PWM + ADC + IO)/TXD3: track 44.5 -> 0.00 mm, vias 2 -> 0
- net /N76E003s (PWM + ADC + IO)/ANA0_1: track 41.3 -> 0.00 mm, vias 2 -> 0
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Other:
- outline, holes or cut-outs redrawn
